Commit message: feat: port Gazebo Sim support from Jazzy to Humble

File: turtlebot3_gazebo/models/turtlebot3_burger/model.sdf.xacro (robot description, xacro)
@@ -1,33 +1,68 @@
 <?xml version="1.0" ?>
-<sdf version="1.8">
-  <model name="turtlebot3_waffle">
-  <pose>0.0 0.0 0.0 0.0 0.0 0.0</pose>
+<sdf version="1.8" xmlns:xacro="http://www.ros.org/wiki/xacro">
+  <xacro:arg
+    name="lds_model"
+    default="$(optenv LDS_MODEL LDS-01)"
+  />
+  <xacro:property
+    name="lds_model_name"
+    value="$(arg lds_model)"
+  />
+  <xacro:property
+    name="lds_min_range"
+    value="${
+      0.12 if lds_model_name == 'LDS-01'
+      else 0.16 if lds_model_name == 'LDS-02'
+      else 0.05 if lds_model_name == 'LDS-03'
+      else 0.12
+    }"
+  />
+  <xacro:property
+    name="lds_max_range"
+    value="${
+      3.5 if lds_model_name == 'LDS-01'
+      else 8.0 if lds_model_name == 'LDS-02'
+      else 12.0 if lds_model_name == 'LDS-03'
+      else 3.5
+    }"
+  />
+  <xacro:property
+    name="lds_update_rate"
+    value="${
+      5.0 if lds_model_name == 'LDS-01'
+      else 5.0 if lds_model_name == 'LDS-02'
+      else 10.0 if lds_model_name == 'LDS-03'
+      else 5.0
+    }"
+  />
+  <model name="turtlebot3_burger">
+    <pose>0.0 0.0 0.0 0.0 0.0 0.0</pose>
     <link name="base_footprint"/>
     <link name="base_link">
       <inertial>
-        <pose>-0.064 0 0.048 0 0 0</pose>
+        <pose>-0.064 0 0.070 0 0 0</pose>
         <inertia>
-          <ixx>4.2111447e-02</ixx>
+          <ixx>1.9527e-02</ixx>
           <ixy>0</ixy>
           <ixz>0</ixz>
-          <iyy>4.2111447e-02</iyy>
+          <iyy>1.9527e-02</iyy>
           <iyz>0</iyz>
-          <izz>7.5254874e-02</izz>
+          <izz>1.9527e-02</izz>
         </inertia>
-        <mass>1.3729096e+00</mass>
+        <mass>8.2573504e-01</mass>
       </inertial>
       <collision name="base_collision">
-        <pose>-0.064 0 0.048 0 0 0</pose>
+        <pose>-0.032 0 0.070 0 0 0</pose>
         <geometry>
           <box>
-            <size>0.265 0.265 0.089</size>
+            <size>0.14 0.14 0.14</size>
           </box>
         </geometry>
       </collision>
       <visual name="base_visual">
-        <pose>-0.064 0 0 0 0 0</pose>
+        <pose>-0.032 0 0 0 0 0</pose>
         <geometry>
           <mesh>
-            <uri>model://turtlebot3_common/meshes/bases/waffle_base.stl</uri>
+            <uri>model://turtlebot3_common/meshes/bases/burger_base.stl</uri>
             <scale>0.001 0.001 0.001</scale>
           </mesh>
@@ -97,17 +132,17 @@
     <link name="base_scan">
       <inertial>
-        <pose>-0.052 0 0.111 0 0 0</pose>
+        <pose>-0.020 0 0.161 0 0 0</pose>
         <inertia>
-          <ixx>0.001</ixx>
+          <ixx>0.0001</ixx>
           <ixy>0.000</ixy>
           <ixz>0.000</ixz>
-          <iyy>0.001</iyy>
+          <iyy>0.0001</iyy>
           <iyz>0.000</iyz>
-          <izz>0.001</izz>
+          <izz>0.0001</izz>
         </inertia>
         <mass>0.114</mass>
       </inertial>
       <collision name="lidar_sensor_collision">
-        <pose>-0.052 0 0.111 0 0 0</pose>
+        <pose>-0.020 0 0.161 0 0 0</pose>
         <geometry>
           <cylinder>
@@ -118,5 +153,5 @@
       </collision>
       <visual name="lidar_sensor_visual">
-        <pose>-0.064 0 0.121 0 0 0</pose>
+        <pose>-0.032 0 0.171 0 0 0</pose>
         <geometry>
           <mesh>
@@ -140,6 +175,6 @@
         <always_on>true</always_on>
         <visualize>true</visualize>
-        <pose>-0.064 0 0.121 0 0 0</pose>
-        <update_rate>10</update_rate>
+        <pose>-0.032 0 0.171 0 0 0</pose>
+        <update_rate>5</update_rate>
         <topic>scan</topic>
         <gz_frame_id>base_scan</gz_frame_id>
@@ -154,6 +189,6 @@
           </scan>
           <range>
-            <min>0.120000</min>
-            <max>3.5</max>
+            <min>${lds_min_range}</min>
+            <max>${lds_max_range}</max>
             <resolution>0.015000</resolution>
           </range>
@@ -168,17 +203,17 @@
     <link name="wheel_left_link">
       <inertial>
-        <pose>0.0 0.144 0.023 -1.57 0 0</pose>
+        <pose>0 0.08 0.023 -1.57 0 0</pose>
         <inertia>
-          <ixx>1.1175580e-05</ixx>
-          <ixy>-4.2369783e-11</ixy>
-          <ixz>-5.9381719e-09</ixz>
-          <iyy>1.1192413e-05</iyy>
-          <iyz>-1.4400107e-11</iyz>
-          <izz>2.0712558e-05</izz>
+          <ixx>5.445e-05</ixx>
+          <ixy>0</ixy>
+          <ixz>0</ixz>
+          <iyy>5.445e-05</iyy>
+          <iyz>0</iyz>
+          <izz>1.089e-04</izz>
         </inertia>
         <mass>0.1</mass>
       </inertial>
       <collision name="wheel_left_collision">
-        <pose>0.0 0.144 0.023 -1.57 0 0</pose>
+        <pose>0 0.08 0.023 -1.57 0 0</pose>
         <geometry>
           <cylinder>
@@ -211,5 +246,5 @@
       </collision>
       <visual name="wheel_left_visual">
-        <pose>0.0 0.144 0.023 0 0 0</pose>
+        <pose>0 0.08 0.023 0 0 0</pose>
         <geometry>
           <mesh>
@@ -233,17 +268,17 @@
     <link name="wheel_right_link">
       <inertial>
-        <pose>0.0 -0.144 0.023 -1.57 0 0</pose>
+        <pose>0.0 -0.08 0.023 -1.57 0 0</pose>
         <inertia>
-          <ixx>1.1175580e-05</ixx>
-          <ixy>-4.2369783e-11</ixy>
-          <ixz>-5.9381719e-09</ixz>
-          <iyy>1.1192413e-05</iyy>
-          <iyz>-1.4400107e-11</iyz>
-          <izz>2.0712558e-05</izz>
+          <ixx>5.445e-05</ixx>
+          <ixy>0</ixy>
+          <ixz>0</ixz>
+          <iyy>5.445e-05</iyy>
+          <iyz>0</iyz>
+          <izz>1.089e-04</izz>
         </inertia>
         <mass>0.1</mass>
       </inertial>
       <collision name="wheel_right_collision">
-        <pose>0.0 -0.144 0.023 -1.57 0 0</pose>
+        <pose>0.0 -0.08 0.023 -1.57 0 0</pose>
         <geometry>
           <cylinder>
@@ -276,5 +311,5 @@
       </collision>
       <visual name="wheel_right_visual">
-        <pose>0.0 -0.144 0.023 0 0 0</pose>
+        <pose>0.0 -0.08 0.023 0 0 0</pose>
         <geometry>
           <mesh>
@@ -296,8 +331,8 @@
       </visual>
     </link>
-    <link name='caster_back_right_link'>
-      <pose>-0.177 -0.064 -0.004 -1.57 0 0</pose>
+    <link name='caster_back_link'>
+      <pose>-0.081 0 -0.004 -1.57 0 0</pose>
       <inertial>
-        <mass>0.001</mass>
+        <mass>0.005</mass>
         <inertia>
           <ixx>0.00001</ixx>
@@ -329,81 +364,4 @@
       </collision>
     </link>
-    <link name='caster_back_left_link'>
-      <pose>-0.177 0.064 -0.004 -1.57 0 0</pose>
-      <inertial>
-        <mass>0.001</mass>
-        <inertia>
-          <ixx>0.00001</ixx>
-          <ixy>0.000</ixy>
-          <ixz>0.000</ixz>
-          <iyy>0.00001</iyy>
-          <iyz>0.000</iyz>
-          <izz>0.00001</izz>
-        </inertia>
-      </inertial>
-      <collision name='collision'>
-        <geometry>
-          <sphere>
-            <radius>0.005000</radius>
-          </sphere>
-        </geometry>
-        <surface>
-          <contact>
-            <ode>
-              <soft_cfm>0</soft_cfm>
-              <soft_erp>0.2</soft_erp>
-              <kp>1e+5</kp>
-              <kd>1</kd>
-              <max_vel>0.01</max_vel>
-              <min_depth>0.001</min_depth>
-            </ode>
-          </contact>
-        </surface>
-      </collision>
-    </link>
-    <link name="camera_link"/>
-    <link name="camera_rgb_frame">
-      <inertial>
-        <pose>0.069 -0.047 0.107 0 0 0</pose>
-        <inertia>
-          <ixx>0.001</ixx>
-          <ixy>0.000</ixy>
-          <ixz>0.000</ixz>
-          <iyy>0.001</iyy>
-          <iyz>0.000</iyz>
-          <izz>0.001</izz>
-        </inertia>
-        <mass>0.035</mass>
-      </inertial>
-      <pose>0.069 -0.047 0.107 0 0 0</pose>
-      <sensor name="camera" type="camera">
-        <always_on>true</always_on>
-        <visualize>true</visualize>
-        <update_rate>30</update_rate>
-        <topic>camera/image_raw</topic>
-        <gz_frame_id>camera_rgb_frame</gz_frame_id>
-        <camera name="intel_realsense_r200">
-          <camera_info_topic>camera/camera_info</camera_info_topic>
-          <horizontal_fov>1.02974</horizontal_fov>
-          <image>
-            <width>1920</width>
-            <height>1080</height>
-            <format>R8G8B8</format>
-          </image>
-          <clip>
-            <near>0.02</near>
-            <far>300</far>
-          </clip>
-          <noise>
-            <type>gaussian</type>
-            <!-- Noise is sampled independently per pixel on each frame.
-                  That pixel's noise value is added to each of its color
-                  channels, which at that point lie in the range [0,1]. -->
-            <mean>0.0</mean>
-            <stddev>0.007</stddev>
-          </noise>
-        </camera>
-      </sensor>
-    </link>
     <joint name="base_joint" type="fixed">
       <parent>base_footprint</parent>
@@ -414,5 +372,5 @@
       <parent>base_link</parent>
       <child>wheel_left_link</child>
-      <pose>0.0 0.144 0.023 -1.57 0 0</pose>
+      <pose>0.0 0.08 0.023 -1.57 0 0</pose>
       <axis>
         <xyz>0 0 1</xyz>
@@ -425,5 +383,5 @@
       <parent>base_link</parent>
       <child>wheel_right_link</child>
-      <pose>0.0 -0.144 0.023 -1.57 0 0</pose>
+      <pose>0.0 -0.08 0.023 -1.57 0 0</pose>
       <axis>
         <xyz>0 0 1</xyz>
@@ -433,11 +391,7 @@
       </axis>
     </joint>
-    <joint name='caster_back_right_joint' type='ball'>
+    <joint name='caster_back_joint' type='ball'>
       <parent>base_link</parent>
-      <child>caster_back_right_link</child>
-    </joint>
-    <joint name='caster_back_left_joint' type='ball'>
-      <parent>base_link</parent>
-      <child>caster_back_left_link</child>
+      <child>caster_back_link</child>
     </joint>
     <joint name="imu_joint" type="fixed">
@@ -452,21 +406,5 @@
       <parent>base_link</parent>
       <child>base_scan</child>
-      <pose>-0.064 0 0.121 0 0 0</pose>
-      <axis>
-        <xyz>0 0 1</xyz>
-      </axis>
-    </joint>
-    <joint name="camera_joint" type="fixed">
-      <parent>base_link</parent>
-      <child>camera_link</child>
-      <pose>0.064 -0.065 0.094 0 0 0</pose>
-      <axis>
-        <xyz>0 0 1</xyz>
-      </axis>
-    </joint>
-    <joint name="camera_rgb_joint" type="fixed">
-      <parent>camera_link</parent>
-      <child>camera_rgb_frame</child>
-      <pose>0.005 0.018 0.013 0 0 0</pose>
+      <pose>-0.032 0 0.171 0 0 0</pose>
       <axis>
         <xyz>0 0 1</xyz>
@@ -478,5 +416,5 @@
       <right_joint>wheel_right_joint</right_joint>
       <!-- kinematics -->
-      <wheel_separation>0.287</wheel_separation>
+      <wheel_separation>0.160</wheel_separation>
       <wheel_radius>0.033</wheel_radius>
       <!-- limits -->

File: turtlebot3_gazebo/models/turtlebot3_burger_cam/model.sdf.xacro (robot description, xacro)
@@ -1,33 +1,68 @@
 <?xml version="1.0" ?>
-<sdf version="1.8">
-  <model name="turtlebot3_waffle">
-  <pose>0.0 0.0 0.0 0.0 0.0 0.0</pose>
+<sdf version="1.8" xmlns:xacro="http://www.ros.org/wiki/xacro">
+  <xacro:arg
+    name="lds_model"
+    default="$(optenv LDS_MODEL LDS-01)"
+  />
+  <xacro:property
+    name="lds_model_name"
+    value="$(arg lds_model)"
+  />
+  <xacro:property
+    name="lds_min_range"
+    value="${
+      0.12 if lds_model_name == 'LDS-01'
+      else 0.16 if lds_model_name == 'LDS-02'
+      else 0.05 if lds_model_name == 'LDS-03'
+      else 0.12
+    }"
+  />
+  <xacro:property
+    name="lds_max_range"
+    value="${
+      3.5 if lds_model_name == 'LDS-01'
+      else 8.0 if lds_model_name == 'LDS-02'
+      else 12.0 if lds_model_name == 'LDS-03'
+      else 3.5
+    }"
+  />
+  <xacro:property
+    name="lds_update_rate"
+    value="${
+      5.0 if lds_model_name == 'LDS-01'
+      else 5.0 if lds_model_name == 'LDS-02'
+      else 10.0 if lds_model_name == 'LDS-03'
+      else 5.0
+    }"
+  />
+  <model name="turtlebot3_burger_cam">
+    <pose>0.0 0.0 0.0 0.0 0.0 0.0</pose>
     <link name="base_footprint"/>
     <link name="base_link">
       <inertial>
-        <pose>-0.064 0 0.048 0 0 0</pose>
-        <inertia>
-          <ixx>4.2111447e-02</ixx>
-          <ixy>0</ixy>
-          <ixz>0</ixz>
-          <iyy>4.2111447e-02</iyy>
-          <iyz>0</iyz>
-          <izz>7.5254874e-02</izz>
-        </inertia>
-        <mass>1.3729096e+00</mass>
+        <pose>-0.032 0 0.070 0 0 0</pose>
+        <inertia>
+          <ixx>7.2397393e-01</ixx>
+          <ixy>4.686399e-10</ixy>
+          <ixz>-1.09525703e-08</ixz>
+          <iyy>7.2397393e-01</iyy>
+          <iyz>2.8582649e-09</iyz>
+          <izz>6.53050163e-01</izz>
+        </inertia>
+        <mass>8.2573504e-01</mass>
       </inertial>
       <collision name="base_collision">
-        <pose>-0.064 0 0.048 0 0 0</pose>
+        <pose>-0.032 0 0.070 0 0 0</pose>
         <geometry>
           <box>
-            <size>0.265 0.265 0.089</size>
+            <size>0.140 0.140 0.140</size>
           </box>
         </geometry>
       </collision>
       <visual name="base_visual">
-        <pose>-0.064 0 0 0 0 0</pose>
+        <pose>-0.032 0 0 0 0 0</pose>
         <geometry>
           <mesh>
-            <uri>model://turtlebot3_common/meshes/bases/waffle_base.stl</uri>
+            <uri>model://turtlebot3_common/meshes/bases/burger_base.stl</uri>
             <scale>0.001 0.001 0.001</scale>
           </mesh>
@@ -97,5 +132,5 @@
     <link name="base_scan">
       <inertial>
-        <pose>-0.052 0 0.111 0 0 0</pose>
+        <pose>-0.020 0 0.161 0 0 0</pose>
         <inertia>
           <ixx>0.001</ixx>
@@ -109,5 +144,5 @@
       </inertial>
       <collision name="lidar_sensor_collision">
-        <pose>-0.052 0 0.111 0 0 0</pose>
+        <pose>-0.020 0 0.161 0 0 0</pose>
         <geometry>
           <cylinder>
@@ -118,5 +153,5 @@
       </collision>
       <visual name="lidar_sensor_visual">
-        <pose>-0.064 0 0.121 0 0 0</pose>
+        <pose>-0.032 0 0.171 0 0 0</pose>
         <geometry>
           <mesh>
@@ -139,7 +174,7 @@
       <sensor name="hls_lfcd_lds" type="gpu_lidar">
         <always_on>true</always_on>
-        <visualize>true</visualize>
-        <pose>-0.064 0 0.121 0 0 0</pose>
-        <update_rate>10</update_rate>
+        <visualize>false</visualize>
+        <pose>-0.032 0 0.171 0 0 0</pose>
+        <update_rate>5</update_rate>
         <topic>scan</topic>
         <gz_frame_id>base_scan</gz_frame_id>
@@ -154,6 +189,6 @@
           </scan>
           <range>
-            <min>0.120000</min>
-            <max>3.5</max>
+            <min>${lds_min_range}</min>
+            <max>${lds_max_range}</max>
             <resolution>0.015000</resolution>
           </range>
@@ -168,17 +203,17 @@
     <link name="wheel_left_link">
       <inertial>
-        <pose>0.0 0.144 0.023 -1.57 0 0</pose>
-        <inertia>
-          <ixx>1.1175580e-05</ixx>
-          <ixy>-4.2369783e-11</ixy>
-          <ixz>-5.9381719e-09</ixz>
-          <iyy>1.1192413e-05</iyy>
-          <iyz>-1.4400107e-11</iyz>
-          <izz>2.0712558e-05</izz>
-        </inertia>
-        <mass>0.1</mass>
+        <pose>0 0.08 0.023 -1.57 0 0</pose>
+        <inertia>
+          <ixx>1.8158194e-03</ixx>
+          <ixy>-9.3392e-12</ixy>
+          <ixz>1.04909e-11</ixz>
+          <iyy>3.2922126e-03</iyy>
+          <iyz>5.75694e-11</iyz>
+          <izz>1.8158194e-03</izz>
+        </inertia>
+        <mass>2.8498940e-02</mass>
       </inertial>
       <collision name="wheel_left_collision">
-        <pose>0.0 0.144 0.023 -1.57 0 0</pose>
+        <pose>0 0.08 0.023 -1.57 0 0</pose>
         <geometry>
           <cylinder>
@@ -211,5 +246,5 @@
       </collision>
       <visual name="wheel_left_visual">
-        <pose>0.0 0.144 0.023 0 0 0</pose>
+        <pose>0 0.08 0.023 0 0 0</pose>
         <geometry>
           <mesh>
@@ -233,17 +268,17 @@
     <link name="wheel_right_link">
       <inertial>
-        <pose>0.0 -0.144 0.023 -1.57 0 0</pose>
-        <inertia>
-          <ixx>1.1175580e-05</ixx>
-          <ixy>-4.2369783e-11</ixy>
-          <ixz>-5.9381719e-09</ixz>
-          <iyy>1.1192413e-05</iyy>
-          <iyz>-1.4400107e-11</iyz>
-          <izz>2.0712558e-05</izz>
-        </inertia>
-        <mass>0.1</mass>
+        <pose>0.0 -0.08 0.023 -1.57 0 0</pose>
+        <inertia>
+          <ixx>1.8158194e-03</ixx>
+          <ixy>-9.3392e-12</ixy>
+          <ixz>1.04909e-11</ixz>
+          <iyy>3.2922126e-03</iyy>
+          <iyz>5.75694e-11</iyz>
+          <izz>1.8158194e-03</izz>
+        </inertia>
+        <mass>2.8498940e-02</mass>
       </inertial>
       <collision name="wheel_right_collision">
-        <pose>0.0 -0.144 0.023 -1.57 0 0</pose>
+        <pose>0.0 -0.08 0.023 -1.57 0 0</pose>
         <geometry>
           <cylinder>
@@ -276,5 +311,5 @@
       </collision>
       <visual name="wheel_right_visual">
-        <pose>0.0 -0.144 0.023 0 0 0</pose>
+        <pose>0.0 -0.08 0.023 0 0 0</pose>
         <geometry>
           <mesh>
@@ -296,15 +331,15 @@
       </visual>
     </link>
-    <link name='caster_back_right_link'>
-      <pose>-0.177 -0.064 -0.004 -1.57 0 0</pose>
-      <inertial>
-        <mass>0.001</mass>
-        <inertia>
-          <ixx>0.00001</ixx>
+    <link name='caster_back_link'>
+      <pose>-0.081 0 -0.004 -1.57 0 0</pose>
+      <inertial>
+        <mass>0.005</mass>
+        <inertia>
+          <ixx>0.001</ixx>
           <ixy>0.000</ixy>
           <ixz>0.000</ixz>
-          <iyy>0.00001</iyy>
+          <iyy>0.001</iyy>
           <iyz>0.000</iyz>
-          <izz>0.00001</izz>
+          <izz>0.001</izz>
         </inertia>
       </inertial>
@@ -329,41 +364,7 @@
       </collision>
     </link>
-    <link name='caster_back_left_link'>
-      <pose>-0.177 0.064 -0.004 -1.57 0 0</pose>
-      <inertial>
-        <mass>0.001</mass>
-        <inertia>
-          <ixx>0.00001</ixx>
-          <ixy>0.000</ixy>
-          <ixz>0.000</ixz>
-          <iyy>0.00001</iyy>
-          <iyz>0.000</iyz>
-          <izz>0.00001</izz>
-        </inertia>
-      </inertial>
-      <collision name='collision'>
-        <geometry>
-          <sphere>
-            <radius>0.005000</radius>
-          </sphere>
-        </geometry>
-        <surface>
-          <contact>
-            <ode>
-              <soft_cfm>0</soft_cfm>
-              <soft_erp>0.2</soft_erp>
-              <kp>1e+5</kp>
-              <kd>1</kd>
-              <max_vel>0.01</max_vel>
-              <min_depth>0.001</min_depth>
-            </ode>
-          </contact>
-        </surface>
-      </collision>
-    </link>
-    <link name="camera_link"/>
-    <link name="camera_rgb_frame">
-      <inertial>
-        <pose>0.069 -0.047 0.107 0 0 0</pose>
+    <link name="camera_link">
+      <inertial>
+        <pose>0.076 0.0 0.093 0 0 0</pose>
         <inertia>
           <ixx>0.001</ixx>
@@ -376,5 +377,5 @@
         <mass>0.035</mass>
       </inertial>
-      <pose>0.069 -0.047 0.107 0 0 0</pose>
+      <pose>0.076 0.0 0.093 0 0 0</pose>
       <sensor name="camera" type="camera">
         <always_on>true</always_on>
@@ -383,15 +384,15 @@
         <topic>camera/image_raw</topic>
         <gz_frame_id>camera_rgb_frame</gz_frame_id>
-        <camera name="intel_realsense_r200">
+        <camera name="picam">
           <camera_info_topic>camera/camera_info</camera_info_topic>
-          <horizontal_fov>1.02974</horizontal_fov>
+          <horizontal_fov>1.085595</horizontal_fov>
           <image>
-            <width>1920</width>
-            <height>1080</height>
-            <format>R8G8B8</format>
+              <width>640</width>
+              <height>480</height>
+              <format>R8G8B8</format>
           </image>
           <clip>
-            <near>0.02</near>
-            <far>300</far>
+              <near>0.03</near>
+              <far>100</far>
           </clip>
           <noise>
@@ -414,5 +415,5 @@
       <parent>base_link</parent>
       <child>wheel_left_link</child>
-      <pose>0.0 0.144 0.023 -1.57 0 0</pose>
+      <pose>0.0 0.08 0.023 -1.57 0 0</pose>
       <axis>
         <xyz>0 0 1</xyz>
@@ -425,5 +426,5 @@
       <parent>base_link</parent>
       <child>wheel_right_link</child>
-      <pose>0.0 -0.144 0.023 -1.57 0 0</pose>
+      <pose>0.0 -0.08 0.023 -1.57 0 0</pose>
       <axis>
         <xyz>0 0 1</xyz>
@@ -433,11 +434,7 @@
       </axis>
     </joint>
-    <joint name='caster_back_right_joint' type='ball'>
-      <parent>base_link</parent>
-      <child>caster_back_right_link</child>
-    </joint>
-    <joint name='caster_back_left_joint' type='ball'>
-      <parent>base_link</parent>
-      <child>caster_back_left_link</child>
+    <joint name='caster_back_joint' type='ball'>
+      <parent>base_link</parent>
+      <child>caster_back_link</child>
     </joint>
     <joint name="imu_joint" type="fixed">
@@ -452,5 +449,5 @@
       <parent>base_link</parent>
       <child>base_scan</child>
-      <pose>-0.064 0 0.121 0 0 0</pose>
+      <pose>-0.032 0 0.171 0 0 0</pose>
       <axis>
         <xyz>0 0 1</xyz>
@@ -460,13 +457,5 @@
       <parent>base_link</parent>
       <child>camera_link</child>
-      <pose>0.064 -0.065 0.094 0 0 0</pose>
-      <axis>
-        <xyz>0 0 1</xyz>
-      </axis>
-    </joint>
-    <joint name="camera_rgb_joint" type="fixed">
-      <parent>camera_link</parent>
-      <child>camera_rgb_frame</child>
-      <pose>0.005 0.018 0.013 0 0 0</pose>
+      <pose>0.040 -0.000 0.110 0 0 0</pose>
       <axis>
         <xyz>0 0 1</xyz>
@@ -478,5 +467,5 @@
       <right_joint>wheel_right_joint</right_joint>
       <!-- kinematics -->
-      <wheel_separation>0.287</wheel_separation>
+      <wheel_separation>0.160</wheel_separation>
       <wheel_radius>0.033</wheel_radius>
       <!-- limits -->
